Commit message: updated urdf

File: IsaacGym_Preview_4_Package/isaacgym/assets/urdf/quadruped.urdf (robot description, URDF)
Before this commit: robot car_robot, 6 links, 5 joints
Joints:
- removed joint joint-base-chassis

File: IsaacGym_Preview_4_Package/isaacgym/assets/urdf/quadruped_v3.urdf (robot description, URDF)
Before this commit: robot car_robot, 10 links, 9 joints
Links:
- link rigid-part-back-left: geometry collision cylinder length=0.02 radius=0.005; visual cylinder length=0.02 radius=0.005
- link rigid-part-back-right: geometry collision cylinder length=0.02 radius=0.005; visual cylinder length=0.02 radius=0.005
- link rigid-part-front-left: geometry collision cylinder length=0.02 radius=0.005; visual cylinder length=0.02 radius=0.005
- link rigid-part-front-right: geometry collision cylinder length=0.02 radius=0.005; visual cylinder length=0.02 radius=0.005
Joints:
- joint joint-base-chassis: type continuous -> fixed
- joint joint-body-rigid-back-left: origin xyz=-0.06 -0.06 0 rpy=0 0 0 -> xyz=-0.08 -0.06 0 rpy=0 0 0
- joint joint-body-rigid-back-right: origin xyz=-0.06 0.06 0 rpy=0 0 0 -> xyz=-0.08 0.11 0 rpy=0 0 0
- joint joint-body-rigid-front-left: origin xyz=0.06 -0.06 0 rpy=0 0 0 -> xyz=0.04 -0.06 0 rpy=0 0 0
- joint joint-body-rigid-front-right: origin xyz=0.06 0.06 0 rpy=0 0 0 -> xyz=0.04 0.11 0 rpy=0 0 0
- joint joint-rigid-back-left-leg: origin xyz=0 0 0 rpy=0 0 0 -> xyz=0 0.02 0 rpy=0 0 0; type continuous -> revolute
- joint joint-rigid-back-right-leg: origin xyz=0 0 0 rpy=0 0 0 -> xyz=0 0.02 0 rpy=0 0 0; type continuous -> revolute
- joint joint-rigid-front-left-leg: origin xyz=0 0 0 rpy=0 0 0 -> xyz=0 0.02 0 rpy=0 0 0; type continuous -> revolute
- joint joint-rigid-front-right-leg: origin xyz=0 0 0 rpy=0 0 0 -> xyz=0 0.02 0 rpy=0 0 0; type continuous -> revolute
